Commit message: noeticで動作確認完了(navigation以外)

File: orne_box_description/urdf/orne_box.urdf.xacro (robot description, xacro)
@@ -45,13 +45,17 @@
   </xacro:wheel_link>
   <!-- Setting for IMU -->
+  <!-- <xacro:sensor_imu name="imu" parent="base_link" size="0.05 0.05 0.05">
+    <origin xyz="0.23 0.0 0.270" rpy="${-PI} 0 ${PI/2}"/>
+  </xacro:sensor_imu> -->
   <xacro:sensor_imu name="imu" parent="base_link" size="0.05 0.05 0.05">
-    <origin xyz="0.23 0.0 0.270" rpy="${-PI} 0 ${PI/2}"/>
+    <origin xyz="-0.04 0.0 0.28" rpy="0 0 0"/>
+    <!-- <origin_child xyz="0.0 0.0 0.0" rpy="0 0 0"/> -->
   </xacro:sensor_imu>
   <!-- Setting for 2D-LiDAR -->
-  <xacro:sensor_hokuyo name="hokuyo" parent="base_link" size="0.05 0.05 0.05">
+  <!-- <xacro:sensor_hokuyo name="hokuyo" parent="base_link" size="0.05 0.05 0.05">
     <origin xyz="0.374295 0 0.2185" rpy="${-PI} 0 0"/>
-  </xacro:sensor_hokuyo>
+  </xacro:sensor_hokuyo> -->
   <xacro:sensor_hokuyo name="mirror_lidar" parent="base_link" size="0.05 0.05 0.05">
-    <origin xyz="-0.08 0.0 0.7" rpy="${-PI} 0.175 0"/>
+    <origin xyz="0.43 0.0 0.34" rpy="0 0.314 0"/>
   </xacro:sensor_hokuyo>
 </robot>

File: orne_box_description/urdf/orne_box_3d_lidar_rfans.urdf.xacro (robot description, xacro)
@@ -8,6 +8,5 @@
     <!-- Setting for 3D-LiDAR -->
     <xacro:VLP-16 parent="base_link" name="surestar" topic="/rfans_points" organize_cloud="false" hz="10" samples="440" gpu="false">
-      <!-- <origin xyz="0.23 0 0.40" rpy="0 0 0"/> -->
-      <origin xyz="-0.105 0 0.80" rpy="0 0 0"/>
+      <origin xyz="0.23 0 0.40" rpy="0 0 3.14"/>
     </xacro:VLP-16>
   </xacro:if>
@@ -15,5 +14,5 @@
     <link name="surestar">
       <inertial>
-        <origin xyz="0.0 0.0 0.0" rpy="0.0 0.0 0.0"/>
+        <origin xyz="0.0 0.0 0.0" rpy="0.0 0.0 3.14"/>
         <mass value="0.3"/>
         <inertia ixx="0.01" ixy="0.0" ixz="0.0" iyy="0.01" iyz="0.0" izz="0.01"/>
