Commit message: update imu

File: orne_box_description/urdf/orne_box3.urdf.xacro (robot description, xacro)
@@ -1,3 +1,3 @@
-<?xml version="1.0" ?>
+<?xml version="1.0"?>
 <robot name="orne_box" xmlns:xacro="http://www.ros.org/wiki/xacro">
   <xacro:property name="PI" value="3.1415926535897931"/>
@@ -167,5 +167,5 @@
   <xacro:include filename="$(find orne_box_description)/urdf/sensors/imu.urdf.xacro"/>
   <xacro:sensor_imu name="imu" parent="base_link" size="0.05 0.05 0.05">
-    <origin xyz="-0.04 0.0 0.28" rpy="0 0 0"/>
+    <origin xyz="-0.04 0.0 0.28" rpy="0 0 ${-PI/2}"/>
   </xacro:sensor_imu>
   <!-- Setting for 2D-LiDAR -->
@@ -182,5 +182,5 @@
   <xacro:include filename="$(find orne_box_description)/urdf/sensors/rfans16.urdf.xacro"/>
   <xacro:sensor_rfans16 name="rfans16" parent="base_link">
-    <origin xyz="-0.105 0 0.40" rpy="0 0 0"/>
+    <origin xyz="-0.105 0 0.80" rpy="0 0 0"/>
   </xacro:sensor_rfans16>
   <transmission name="tran1">
