Commit message: update

File: orne_box_description/urdf/orne_box_3d_lidar.urdf.xacro (robot description, xacro)
@@ -9,5 +9,5 @@
     <xacro:VLP-16 parent="base_link" name="surestar" topic="/rfans_points" organize_cloud="false" hz="10" samples="440" gpu="false">
       <!-- <origin xyz="0.23 0 0.40" rpy="0 0 0"/> -->
-      <origin xyz="-0.105 0 0.80" rpy="0 0 0"/>
+      <origin xyz="-0.12 0 0.60" rpy="0 0 0"/>
     </xacro:VLP-16>
   </xacro:if>

File: orne_box_description/urdf/orne_box_3d_lidar_rfans.urdf.xacro (robot description, xacro)
@@ -8,5 +8,5 @@
     <!-- Setting for 3D-LiDAR -->
     <xacro:VLP-16 parent="base_link" name="surestar" topic="/rfans_points" organize_cloud="false" hz="10" samples="440" gpu="false">
-      <origin xyz="0.23 0 0.40" rpy="0 0 3.14"/>
+      <origin xyz="-0.12 0 0.60" rpy="0 0 0"/>
     </xacro:VLP-16>
   </xacro:if>
@@ -14,5 +14,5 @@
     <link name="surestar">
       <inertial>
-        <origin xyz="0.0 0.0 0.0" rpy="0.0 0.0 3.14"/>
+        <origin xyz="0.0 0.0 0.0" rpy="0.0 0.0 0"/>
         <mass value="0.3"/>
         <inertia ixx="0.01" ixy="0.0" ixz="0.0" iyy="0.01" iyz="0.0" izz="0.01"/>
@@ -33,5 +33,5 @@
     </link>
     <joint name="surestar_joint" type="fixed">
-      <origin xyz="0.23 0.0 0.4" rpy="0.0 0.0 0.0"/>
+      <origin xyz="-0.12 0.0 0.6" rpy="0.0 0.0 0.0"/>
       <parent link="base_link"/>
       <child link="surestar"/>
@@ -73,5 +73,5 @@
     </gazebo>
   </xacro:if>
-  <xacro:include filename="$(find orne_box_description)/urdf/sensors/gnss.urdf.xacro"/> -->
+  <xacro:include filename="$(find orne_box_description)/urdf/sensors/gnss.urdf.xacro"/>
   <xacro:include filename="$(find orne_box_description)/urdf/sensors/camera.urdf.xacro"/>
   <xacro:sensor_gnss name="gnss" parent="base_link">

Commit message: ミラーLiDAR用のurdfを作成

File: orne_box_description/urdf/orne_box_3d_lidar.urdf.xacro (robot description, xacro)
@@ -74,5 +74,6 @@
     </gazebo>
   </xacro:if>
-  <!-- <xacro:include filename="$(find orne_box_description)/urdf/sensors/gnss.urdf.xacro"/>
+<!--
+  <xacro:include filename="$(find orne_box_description)/urdf/sensors/gnss.urdf.xacro"/>
   <xacro:include filename="$(find orne_box_description)/urdf/sensors/camera.urdf.xacro"/>
   <xacro:sensor_gnss name="gnss" parent="base_link">
@@ -80,5 +81,6 @@
   </xacro:sensor_gnss>
   <xacro:sensor_camera name="camera" parent="base_link">
-    <origin xyz="-0.08 0.0 0.8" rpy="0 0.38 0"/>
-  </xacro:sensor_camera> -->
+    <origin xyz="-0.12 0.0 0.8" rpy="0 0.38 0"/>
+  </xacro:sensor_camera>
+  -->
 </robot>

File: orne_box_description/urdf/orne_box_3d_lidar_rfans.urdf.xacro (robot description, xacro)
@@ -1,81 +1,20 @@
 <?xml version="1.0"?>
 <robot xmlns:xacro="http://www.ros.org/wiki/xacro" name="orne_box">
-  <xacro:arg name="ignition_gazebo" default="false"/>
+  <!-- 元のファイルのインクルード -->
   <xacro:include filename="$(find orne_box_description)/urdf/orne_box.urdf.xacro"/>
-  <!-- @TODO More clear boolean operation -->
-  <xacro:if value="${'$(arg ignition_gazebo)' == 'false'}">
-    <xacro:include filename="$(find velodyne_description)/urdf/VLP-16.urdf.xacro"/>
-    <!-- Setting for 3D-LiDAR -->
-    <xacro:VLP-16 parent="base_link" name="surestar" topic="/rfans_points" organize_cloud="false" hz="10" samples="440" gpu="false">
-      <origin xyz="-0.12 0 0.60" rpy="0 0 0"/>
-    </xacro:VLP-16>
-  </xacro:if>
-  <xacro:if value="$(arg ignition_gazebo)">
-    <link name="surestar">
-      <inertial>
-        <origin xyz="0.0 0.0 0.0" rpy="0.0 0.0 0"/>
-        <mass value="0.3"/>
-        <inertia ixx="0.01" ixy="0.0" ixz="0.0" iyy="0.01" iyz="0.0" izz="0.01"/>
-      </inertial>
-      <visual name="surestar_visual">
-        <origin xyz="0.0 0.0 0.0" rpy="0.0 0.0 0.0"/>
-        <geometry>
-          <cylinder radius="0.06" length="0.1"/>
-        </geometry>
-        <material name="green"/>
-      </visual>
-      <collision name="surestar_collision">
-        <origin xyz="0.0 0.0 0.0" rpy="0.0 0.0 0.0"/>
-        <geometry>
-          <cylinder radius="0.06" length="0.13"/>
-        </geometry>
-      </collision>
-    </link>
-    <joint name="surestar_joint" type="fixed">
-      <origin xyz="-0.12 0.0 0.6" rpy="0.0 0.0 0.0"/>
-      <parent link="base_link"/>
-      <child link="surestar"/>
-    </joint>
-    <gazebo reference="surestar">
-      <sensor name="surestar" type="gpu_lidar">
-        <alwaysOn>1</alwaysOn>
-        <update_rate>10</update_rate>
-        <visualize>true</visualize>
-        <lidar>
-          <scan>
-            <horizontal>
-              <!-- Correct points of 1875 -->
-              <samples>722</samples>
-              <resolution>1</resolution>
-              <min_angle>-3.141592</min_angle>
-              <max_angle>3.141592</max_angle>
-            </horizontal>
-            <vertical>
-              <samples>16</samples>
-              <resolution>1</resolution>
-              <min_angle>-0.261799</min_angle>
-              <max_angle>0.261799</max_angle>
-            </vertical>
-          </scan>
-          <range>
-            <min>0.3</min>
-            <max>100.0</max>
-            <resolution>0.001</resolution>
-          </range>
-          <noise>
-            <noise>gaussian</noise>
-            <mean>0.0</mean>
-            <stddev>0.02</stddev>
-          </noise>
-        </lidar>
-        <topic>model/orne_box/rfans</topic>
-      </sensor>
-    </gazebo>
-  </xacro:if>
+  <!-- RFans-16のインクルード -->
+  <xacro:include filename="$(find orne_box_description)/urdf/sensors/rfans.urdf.xacro"/>
+  <!-- GNSSとカメラのインクルード -->
   <xacro:include filename="$(find orne_box_description)/urdf/sensors/gnss.urdf.xacro"/>
   <xacro:include filename="$(find orne_box_description)/urdf/sensors/camera.urdf.xacro"/>
+  <!-- RFans-16センサー設定 -->
+  <xacro:VLP-16 name="surestar" parent="base_link" topic="/rfans_points" organize_cloud="false" hz="10" samples="440" gpu="false">
+    <origin xyz="-0.12 0.0 0.60" rpy="0 0 0"/>
+  </xacro:VLP-16>
+  <!-- GNSSセンサー設定 -->
   <xacro:sensor_gnss name="gnss" parent="base_link">
     <origin xyz="-0.12 0.12 0.9" rpy="0 0 0"/>
   </xacro:sensor_gnss>
+  <!-- カメラセンサー設定 -->
   <xacro:sensor_camera name="camera" parent="base_link">
     <origin xyz="-0.08 0.0 0.8" rpy="0 0.38 0"/>
